File: Flash_JTAG.kicad_sch (KiCad schematic)
At the start: 48 parts, among them J1 USB Type C, Q1 MMST2222A, SW1 User, U1 LFE5U-85F-8BG381C, U2 IS25LP128F, U3 FT231XQ, Y1 50MHz

Commit message: Switched to project library
Parts:
- F1: footprint Gil:Fuse_1812_4532Metric -> ECP5_RISCV:Fuse_1812_4532Metric
- J1: footprint Gil:USB_C_Receptacle_GCT_USB4105-xx-A_16P_TopMnt_Horizontal -> ECP5_RISCV:USB_C_Receptacle_GCT_USB4105-xx-A_16P_TopMnt_Horizontal; symbol Gil:USB_C_Receptacle_USB2.0 -> ECP5_RISCV:USB_C_Receptacle_USB2.0
- U1: footprint Gil:BGA-381_pitch0.8mm_dia0.4mm -> ECP5_RISCV:BGA-381_pitch0.8mm_dia0.4mm; symbol Gil:LFE5U-85F-6BG381x -> ECP5_RISCV:LFE5U-85F-6BG381x
- U2: footprint Gil:WSON-8-1EP_6x5mm_P1.27mm_EP3.4x4.3mm -> ECP5_RISCV:WSON-8-1EP_6x5mm_P1.27mm_EP3.4x4.3mm; symbol Memory_EEPROM:25LCxxx -> ECP5_RISCV:25LCxxx
- U3: symbol Gil:FT231XQ -> ECP5_RISCV:FT231XQ
- Y1: footprint Gil:Oscillator_SMD_Diodes_FN-4Pin_7.0x5.0mm -> ECP5_RISCV:Oscillator_SMD_Diodes_FN-4Pin_7.0x5.0mm

Commit message: Changed the name of the project path to ECP5_BGA381_RISCV
Parts:
- F1: footprint ECP5_RISCV:Fuse_1812_4532Metric -> ECP5_BGA381_RISCV:Fuse_1812_4532Metric
- J1: footprint ECP5_RISCV:USB_C_Receptacle_GCT_USB4105-xx-A_16P_TopMnt_Horizontal -> ECP5_BGA381_RISCV:USB_C_Receptacle_GCT_USB4105-xx-A_16P_TopMnt_Horizontal; symbol ECP5_RISCV:USB_C_Receptacle_USB2.0 -> ECP5_BGA381_RISCV:USB_C_Receptacle_USB2.0
- U1: footprint ECP5_RISCV:BGA-381_pitch0.8mm_dia0.4mm -> ECP5_BGA381_RISCV:BGA-381_pitch0.8mm_dia0.4mm; symbol ECP5_RISCV:LFE5U-85F-6BG381x -> ECP5_BGA381_RISCV:LFE5U-85F-6BG381x
- U2: footprint ECP5_RISCV:WSON-8-1EP_6x5mm_P1.27mm_EP3.4x4.3mm -> ECP5_BGA381_RISCV:WSON-8-1EP_6x5mm_P1.27mm_EP3.4x4.3mm; symbol ECP5_RISCV:25LCxxx -> ECP5_BGA381_RISCV:25LCxxx
- U3: symbol ECP5_RISCV:FT231XQ -> ECP5_BGA381_RISCV:FT231XQ
- Y1: footprint ECP5_RISCV:Oscillator_SMD_Diodes_FN-4Pin_7.0x5.0mm -> ECP5_BGA381_RISCV:Oscillator_SMD_Diodes_FN-4Pin_7.0x5.0mm
Changed lines of the file:
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@@
 	)
 	(symbol
-		(lib_id "ECP5_RISCV:FT231XQ")
+		(lib_id "ECP5_BGA381_RISCV:FT231XQ")
 		(at 101.6 139.7 0)
 		(unit 1)
@@
 			)
 		)
-		(property "Footprint" "ECP5_RISCV:Oscillator_SMD_Diodes_FN-4Pin_7.0x5.0mm"
+		(property "Footprint" "ECP5_BGA381_RISCV:Oscillator_SMD_Diodes_FN-4Pin_7.0x5.0mm"
 			(at 256.54 133.35 0)
 			(effects
@@
 	)
 	(symbol
-		(lib_id "ECP5_RISCV:USB_C_Receptacle_USB2.0")
+		(lib_id "ECP5_BGA381_RISCV:USB_C_Receptacle_USB2.0")
 		(at 34.29 132.08 0)
 		(unit 1)
@@
 			)
 		)
-		(property "Footprint" "ECP5_RISCV:USB_C_Receptacle_GCT_USB4105-xx-A_16P_TopMnt_Horizontal"
+		(property "Footprint" "ECP5_BGA381_RISCV:USB_C_Receptacle_GCT_USB4105-xx-A_16P_TopMnt_Horizontal"
 			(at 38.1 132.08 0)
 			(effects
@@
 	)
 	(symbol
-		(lib_id "ECP5_RISCV:LFE5U-85F-6BG381x")
+		(lib_id "ECP5_BGA381_RISCV:LFE5U-85F-6BG381x")
 		(at 135.89 45.72 0)
 		(unit 8)
@@
 			)
 		)
-		(property "Footprint" "ECP5_RISCV:BGA-381_pitch0.8mm_dia0.4mm"
+		(property "Footprint" "ECP5_BGA381_RISCV:BGA-381_pitch0.8mm_dia0.4mm"
 			(at 132.08 -111.76 0)
 			(effects
@@
 	)
 	(symbol
-		(lib_id "ECP5_RISCV:LFE5U-85F-6BG381x")
+		(lib_id "ECP5_BGA381_RISCV:LFE5U-85F-6BG381x")
 		(at 240.03 64.77 0)
 		(unit 3)
@@
 			)
 		)
-		(property "Footprint" "ECP5_RISCV:BGA-381_pitch0.8mm_dia0.4mm"
+		(property "Footprint" "ECP5_BGA381_RISCV:BGA-381_pitch0.8mm_dia0.4mm"
 			(at 236.22 -92.71 0)
 			(effects
@@
 	)
 	(symbol
-		(lib_id "ECP5_RISCV:25LCxxx")
+		(lib_id "ECP5_BGA381_RISCV:25LCxxx")
 		(at 41.91 71.12 0)
 		(unit 1)
@@
 			)
 		)
-		(property "Footprint" "ECP5_RISCV:WSON-8-1EP_6x5mm_P1.27mm_EP3.4x4.3mm"
+		(property "Footprint" "ECP5_BGA381_RISCV:WSON-8-1EP_6x5mm_P1.27mm_EP3.4x4.3mm"
 			(at 41.91 71.12 0)
 			(effects
@@
 	)
 	(symbol
-		(lib_id "ECP5_RISCV:LFE5U-85F-6BG381x")
+		(lib_id "ECP5_BGA381_RISCV:LFE5U-85F-6BG381x")
 		(at 279.4 64.77 0)
 		(unit 6)
@@
 			)
 		)
-		(property "Footprint" "ECP5_RISCV:BGA-381_pitch0.8mm_dia0.4mm"
+		(property "Footprint" "ECP5_BGA381_RISCV:BGA-381_pitch0.8mm_dia0.4mm"
 			(at 275.59 -92.71 0)
 			(effects
@@
 			)
 		)
-		(property "Footprint" "ECP5_RISCV:Fuse_1812_4532Metric"
+		(property "Footprint" "ECP5_BGA381_RISCV:Fuse_1812_4532Metric"
 			(at 55.88 118.11 0)
 			(effects
@@
 	)
 	(symbol
-		(lib_id "ECP5_RISCV:LFE5U-85F-6BG381x")
+		(lib_id "ECP5_BGA381_RISCV:LFE5U-85F-6BG381x")
 		(at 175.26 113.03 0)
 		(mirror y)
@@
 			)
 		)
-		(property "Footprint" "ECP5_RISCV:BGA-381_pitch0.8mm_dia0.4mm"
+		(property "Footprint" "ECP5_BGA381_RISCV:BGA-381_pitch0.8mm_dia0.4mm"
 			(at 179.07 -44.45 0)
 			(effects
