File: Power.kicad_sch (KiCad schematic)
At the start: 42 parts, among them U1 LFE5U-85F-8BG381C, U5 TLV62569DBVT, U6 TLV62569DBVT, U7 TLV62569DBVT

Commit message: Switched to project library
Parts:
- U1: footprint Gil:BGA-381_pitch0.8mm_dia0.4mm -> ECP5_RISCV:BGA-381_pitch0.8mm_dia0.4mm; symbol Gil:LFE5U-85F-6BG381x -> ECP5_RISCV:LFE5U-85F-6BG381x

Commit message: Changed the name of the project path to ECP5_BGA381_RISCV
Parts:
- U1: footprint ECP5_RISCV:BGA-381_pitch0.8mm_dia0.4mm -> ECP5_BGA381_RISCV:BGA-381_pitch0.8mm_dia0.4mm; symbol ECP5_RISCV:LFE5U-85F-6BG381x -> ECP5_BGA381_RISCV:LFE5U-85F-6BG381x
Changed lines of the file:
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@@
 	)
 	(symbol
-		(lib_id "ECP5_RISCV:LFE5U-85F-6BG381x")
+		(lib_id "ECP5_BGA381_RISCV:LFE5U-85F-6BG381x")
 		(at 92.71 107.95 0)
 		(unit 1)
@@
 			)
 		)
-		(property "Footprint" "ECP5_RISCV:BGA-381_pitch0.8mm_dia0.4mm"
+		(property "Footprint" "ECP5_BGA381_RISCV:BGA-381_pitch0.8mm_dia0.4mm"
 			(at 88.9 -49.53 0)
 			(effects
